File: PCB/kicad/powerline.sch (KiCad schematic (older format))
At the start: 22 parts

Commit message: Moved PCB files
Other:
- note removed: "Relay0"
Changed lines of the file:
@@
 	1    0    0    -1
 $EndComp
-Text Notes 6400 3550 0    50   ~ 0
-Relay0
 Text Notes 6400 1350 0    50   ~ 0
 RELAY1
